File: 1bitsy/v1.0b/1bitsy.sch (KiCad schematic (older format))
At the start: 87 parts, among them J1 BOOT, P1 CONN_01X01, P10 CONN_01X01, P11 CONN_01X01, P12 CONN_01X01, P13 CONN_01X01, P14 CONN_01X01, P15 CONN_01X01, P16 CONN_01X01, P17 CONN_01X01, P18 CONN_01X01, P19 CONN_01X01, P2 CONN_01X01, P20 CONN_01X01, P21 CONN_01X01, P22 CONN_01X01, P23 CONN_01X01, P24 USB_OTG, P25 CONN_01X01, P26 CONN_01X01, P27 CONN_01X01, P28 CONN_01X01, P29 CONN_01X01, P3 CONN_01X01, P30 CONN_01X01, P31 CONN_01X01, P32 CONN_01X01, P33 CONN_01X01, P34 CONN_01X01, P35 CONN_01X01, P36 CONN_01X01, P37 CONN_01X01, P38 CONN_01X01, P39 CONN_01X01, P4 CONN_01X01, P40 CONN_01X01, P41 CONN_01X01, P42 CONN_01X01, P43 CONN_01X01, P44 CONN_01X01, P45 CONN_01X01, P46 CONN_01X01, P47 CONN_01X01, P48 CONN_01X01, P49 CONN_01X01, P5 CONN_01X01, P50 CONN_01X01, P51 CONN_01X01, P52 CONN_01X01, P6 CONN_01X01, P7 CONN_01X01, P8 CONN_01X01, P9 CONN_01X01, SW1 TACT_G, U1 VREG_3V3, U2 STM32F415RGT, X1 32.768kHz, X2 25MHz, X3 JTAG-10

Commit message: First routing pass on 1BitSy V1.0b.
Parts:
- removed P43, P44, P45, P46, P47: CONN_01X01, pkl_pads:PAD_SMD_R_1x1, symbol CONN_01X01
- added P43, P44, P45, P46, P47: TP, pkl_pads:POGO_PAD_SMD_R_1x1, symbol POGO_PAD_SMD
- added P54, P55: CONN_01X01, pkl_pin_headers:Pin_Header_Straight_Round_1x01, symbol CONN_01X01
- X1: footprint Crystals:Crystal_Round_Horizontal_2mm -> pkl_misc:ABS07
- gave numbers to parts that had none: 1
Connections:
- net +3V3: now also P54.1 (P1); no longer U2.1 (VBAT)
- net GND: now also P55.1 (P1)
- net JTAG_RST: now also P47.1 (PAD)
- net JTAG_TCK: now also P44.1 (PAD)
- net JTAG_TDI: now also P46.1 (PAD)
- net JTAG_TDO: now also P45.1 (PAD)
- net JTAG_TMS: now also P43.1 (PAD)
- net VBAT: now reaches P53.1 (P1)
- net VBAT: now also U2.1 (VBAT)
Other:
- moved on the sheet: P40, P41, P42, P53
