File: 1bitsy/v1.0b/1bitsy.kicad_pcb (KiCad board)
At the start: 4 copper layers, 38.1 x 17.8 mm, 98 parts, among them J1 BOOT, P1 CONN_01X01, P10 CONN_01X01, P11 CONN_01X01, P12 CONN_01X01, P13 CONN_01X01, P14 CONN_01X01, P15 CONN_01X01, P16 CONN_01X01, P17 CONN_01X01, P18 CONN_01X01, P19 CONN_01X01, P2 CONN_01X01, P20 CONN_01X01, P21 CONN_01X01, P22 CONN_01X01, P23 CONN_01X01, P24 USB_OTG, P25 CONN_01X01, P26 CONN_01X01, P27 CONN_01X01, P28 CONN_01X01, P29 CONN_01X01, P3 CONN_01X01, P30 CONN_01X01, P31 CONN_01X01, P32 CONN_01X01, P33 CONN_01X01, P34 CONN_01X01, P35 CONN_01X01, P36 CONN_01X01, P37 CONN_01X01, P38 CONN_01X01, P39 CONN_01X01, P4 CONN_01X01, P40 CONN_01X01, P41 CONN_01X01, P42 CONN_01X01, P43 TP, P44 TP, P45 TP, P46 TP, P47 TP, P48 CONN_01X01, P49 CONN_01X01, P5 CONN_01X01, P50 CONN_01X01, P51 CONN_01X01, P52 CONN_01X01, P53 CONN_01X01, P54 CONN_01X01, P55 CONN_01X01, P6 CONN_01X01, P7 CONN_01X01, P8 CONN_01X01, P9 CONN_01X01, SW1 TACT_G, U1 VREG_3V3, U2 STM32F415RGT, X1 32.768kHz, X2 25MHz, X3 JTAG-10

Commit message: Made the legend split line split.
Parts:
- added REF**: via0305, pkl_misc:via0305, F.Cu at (135.9, 39.4)
Changed lines of the file:
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@@
     (links 152)
     (no_connects 0)
-    (area 96.542667 26.87 157.365715 59.364)
+    (area 100.254999 36.744999 138.505001 54.695001)
     (thickness 1.6)
-    (drawings 333)
+    (drawings 367)
     (tracks 793)
     (zones 0)
-    (modules 98)
+    (modules 99)
     (nets 64)
   )
@@
   )
   (module pkl_misc:via0305 (layer F.Cu)
+    (at 135.88 39.37)
+    (fp_text reference REF** (at 0 0.35) (layer F.SilkS) hide
+      (effects (font (size 0.127 0.127) (thickness 0.03175)))
+    )
+    (fp_text value via0305 (at 0 -0.35) (layer F.Fab) hide
+      (effects (font (size 0.127 0.127) (thickness 0.03175)))
+    )
+    (pad 1 thru_hole circle (at 0 0) (size 0.5 0.5) (drill 0.3) (layers *.Cu)
+      (net 2 GND) (zone_connect 2))
+  )
+  (module pkl_misc:via0305 (layer F.Cu)
     (at 119.23 45.37)
     (fp_text reference REF** (at 0 0.35) (layer F.SilkS) hide
@@
       (net 2 GND) (zone_connect 2))
   )
+  (gr_line (start 137.18 51.695) (end 137.18 52.07) (layer F.SilkS) (width 0.15))
+  (gr_line (start 137.18 49.145) (end 137.18 49.92) (layer F.SilkS) (width 0.15))
+  (gr_line (start 137.18 46.62) (end 137.18 47.37) (layer F.SilkS) (width 0.15))
+  (gr_line (start 137.18 44.07) (end 137.18 44.82) (layer F.SilkS) (width 0.15))
+  (gr_line (start 137.18 41.545) (end 137.18 42.295) (layer F.SilkS) (width 0.15))
+  (gr_line (start 137.18 39.37) (end 137.18 39.745) (layer F.SilkS) (width 0.15))
+  (gr_line (start 134.63 39.745) (end 134.63 39.37) (layer F.SilkS) (width 0.15))
+  (gr_line (start 134.63 42.295) (end 134.63 41.545) (layer F.SilkS) (width 0.15))
+  (gr_line (start 134.63 44.82) (end 134.63 44.07) (layer F.SilkS) (width 0.15))
+  (gr_line (start 134.63 47.37) (end 134.63 46.62) (layer F.SilkS) (width 0.15))
+  (gr_line (start 134.63 49.92) (end 134.63 49.145) (layer F.SilkS) (width 0.15))
+  (gr_line (start 134.63 52.07) (end 134.63 51.695) (layer F.SilkS) (width 0.15))
+  (gr_line (start 103.23 53.37) (end 102.88 53.37) (layer F.SilkS) (width 0.15))
+  (gr_line (start 105.78 53.37) (end 105.03 53.37) (layer F.SilkS) (width 0.15))
+  (gr_line (start 108.33 53.37) (end 107.58 53.37) (layer F.SilkS) (width 0.15))
+  (gr_line (start 110.88 53.37) (end 110.105 53.37) (layer F.SilkS) (width 0.15))
+  (gr_line (start 113.405 53.37) (end 112.655 53.37) (layer F.SilkS) (width 0.15))
+  (gr_line (start 115.955 53.37) (end 115.18 53.37) (layer F.SilkS) (width 0.15))
+  (gr_line (start 118.48 53.37) (end 117.73 53.37) (layer F.SilkS) (width 0.15))
+  (gr_line (start 121.03 53.37) (end 120.28 53.37) (layer F.SilkS) (width 0.15))
+  (gr_line (start 123.555 53.37) (end 122.805 53.37) (layer F.SilkS) (width 0.15))
+  (gr_line (start 126.105 53.37) (end 125.355 53.37) (layer F.SilkS) (width 0.15))
+  (gr_line (start 128.655 53.37) (end 127.88 53.37) (layer F.SilkS) (width 0.15))
+  (gr_line (start 131.18 53.37) (end 130.43 53.37) (layer F.SilkS) (width 0.15))
+  (gr_line (start 133.33 53.37) (end 132.98 53.37) (layer F.SilkS) (width 0.15))
+  (gr_line (start 105.78 38.12) (end 105.43 38.12) (layer F.SilkS) (width 0.15))
+  (gr_line (start 108.33 38.12) (end 107.58 38.12) (layer F.SilkS) (width 0.15))
+  (gr_line (start 110.88 38.12) (end 110.105 38.12) (layer F.SilkS) (width 0.15))
+  (gr_line (start 113.405 38.12) (end 112.655 38.12) (layer F.SilkS) (width 0.15))
+  (gr_line (start 115.955 38.12) (end 115.18 38.12) (layer F.SilkS) (width 0.15))
+  (gr_line (start 118.48 38.12) (end 117.73 38.12) (layer F.SilkS) (width 0.15))
+  (gr_line (start 121.03 38.12) (end 120.28 38.12) (layer F.SilkS) (width 0.15))
+  (gr_line (start 123.58 38.12) (end 122.805 38.12) (layer F.SilkS) (width 0.15))
+  (gr_line (start 126.105 38.12) (end 125.355 38.12) (layer F.SilkS) (width 0.15))
+  (gr_line (start 128.655 38.12) (end 127.88 38.12) (layer F.SilkS) (width 0.15))
+  (gr_line (start 131.18 38.12) (end 130.43 38.12) (layer F.SilkS) (width 0.15))
+  (gr_line (start 133.73 38.12) (end 132.98 38.12) (layer F.SilkS) (width 0.15))
+  (gr_line (start 135.505 38.12) (end 135.88 38.12) (layer F.SilkS) (width 0.15))
   (gr_text 9 (at 107.58 37.37 315) (layer F.SilkS)
     (effects (font (size 0.5 0.5) (thickness 0.125)))
@@
     (effects (font (size 0.5 0.5) (thickness 0.125)))
   )
-  (gr_line (start 135.88 38.12) (end 105.43 38.12) (layer F.SilkS) (width 0.15))
   (gr_text D (at 136.355 37.295 45) (layer F.SilkS)
     (effects (font (size 0.5 0.5) (thickness 0.125)))
@@
     (effects (font (size 0.5 0.5) (thickness 0.125)))
   )
-  (gr_line (start 137.18 39.37) (end 137.18 52.07) (layer F.SilkS) (width 0.15))
-  (gr_line (start 134.63 39.37) (end 134.63 52.07) (layer F.SilkS) (width 0.15))
-  (gr_line (start 133.33 53.37) (end 102.88 53.37) (layer F.SilkS) (width 0.15))
   (gr_text 3 (at 131.23 54.12 135) (layer F.SilkS)
     (effects (font (size 0.5 0.5) (thickness 0.125)))

Commit message: Improved part ID and Value legend.
Parts:
- L1: value 600 Ferrite -> Ferr
