File: 1bitsy/v1.0d/1bitsy-rr.kicad_pcb (KiCad board)
At the start: 4 copper layers, 38.1 x 17.8 mm, 108 parts, among them J1 BOOT, P1 CONN_01X01, P10 CONN_01X01, P11 CONN_01X01, P12 CONN_01X01, P13 CONN_01X01, P14 CONN_01X01, P15 CONN_01X01, P16 CONN_01X01, P17 CONN_01X01, P18 CONN_01X01, P19 CONN_01X01, P2 CONN_01X01, P20 CONN_01X01, P21 CONN_01X01, P22 CONN_01X01, P23 CONN_01X01, P24 USB_OTG, P25 CONN_01X01, P26 CONN_01X01, P27 CONN_01X01, P28 CONN_01X01, P29 CONN_01X01, P3 CONN_01X01, P30 CONN_01X01, P31 CONN_01X01, P32 CONN_01X01, P33 CONN_01X01, P34 CONN_01X01, P35 CONN_01X01, P36 CONN_01X01, P37 CONN_01X01, P38 CONN_01X01, P39 CONN_01X01, P4 CONN_01X01, P40 CONN_01X01, P41 CONN_01X01, P42 CONN_01X01, P43 TP, P44 TP, P45 TP, P46 TP, P47 TP, P48 CONN_01X01, P49 CONN_01X01, P5 CONN_01X01, P50 CONN_01X01, P51 CONN_01X01, P52 CONN_01X01, P53 CONN_01X01, P54 CONN_01X01, P55 CONN_01X01, P6 CONN_01X01, P7 CONN_01X01, P8 CONN_01X01, P9 CONN_01X01, SW1 TACT_G, U1 VREG_3V3, U2 STM32F415RGT, X1 32.768kHz, X2 25MHz, X3 JTAG-10

Commit message: Fixed the LS crystal label.
We had 36KHz but should be 32KHz if anything. (yes we are truncating the
actual frequency because we lack space for all the stuff behind the
comma)
Other:
- board text added: "RTC 32KHz"
- board text removed: "RTC 36KHz"
Changed lines of the file:
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@@
     (links 160)
     (no_connects 0)
-    (area 100.279999 36.769999 138.480001 54.670001)
+    (area 90.322667 29.02 150.365716 59.4815)
     (thickness 1.6)
     (drawings 336)
@@
     (effects (font (size 0.9 0.9) (thickness 0.2)) (justify mirror))
   )
-  (gr_text "RTC 36KHz" (at 123.53 45.72 90) (layer B.SilkS)
+  (gr_text "RTC 32KHz" (at 123.53 45.72 90) (layer B.SilkS)
     (effects (font (size 0.5 0.5) (thickness 0.125)) (justify mirror))
   )
