File: 1bitsy/v1.0d/1bitsy.kicad_pcb (KiCad board)
At the start: 4 copper layers, 38.1 x 17.8 mm, 108 parts, among them J1 BOOT, P1 CONN_01X01, P10 CONN_01X01, P11 CONN_01X01, P12 CONN_01X01, P13 CONN_01X01, P14 CONN_01X01, P15 CONN_01X01, P16 CONN_01X01, P17 CONN_01X01, P18 CONN_01X01, P19 CONN_01X01, P2 CONN_01X01, P20 CONN_01X01, P21 CONN_01X01, P22 CONN_01X01, P23 CONN_01X01, P24 USB_OTG, P25 CONN_01X01, P26 CONN_01X01, P27 CONN_01X01, P28 CONN_01X01, P29 CONN_01X01, P3 CONN_01X01, P30 CONN_01X01, P31 CONN_01X01, P32 CONN_01X01, P33 CONN_01X01, P34 CONN_01X01, P35 CONN_01X01, P36 CONN_01X01, P37 CONN_01X01, P38 CONN_01X01, P39 CONN_01X01, P4 CONN_01X01, P40 CONN_01X01, P41 CONN_01X01, P42 CONN_01X01, P43 TP, P44 TP, P45 TP, P46 TP, P47 TP, P48 CONN_01X01, P49 CONN_01X01, P5 CONN_01X01, P50 CONN_01X01, P51 CONN_01X01, P52 CONN_01X01, P53 CONN_01X01, P54 CONN_01X01, P55 CONN_01X01, P6 CONN_01X01, P7 CONN_01X01, P8 CONN_01X01, P9 CONN_01X01, SW1 TACT_G, U1 VREG_3V3, U2 STM32F415RGT, X1 32.768kHz, X2 25MHz, X3 JTAG-10

Commit message: Fixed the LS crystal label.
We had 36KHz but should be 32KHz if anything. (yes we are truncating the
actual frequency because we lack space for all the stuff behind the
comma)
Other:
- board text added: "RTC 32KHz"
- board text removed: "RTC 36KHz"
Changed lines of the file:
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@@
-(kicad_pcb (version 4) (host pcbnew 4.0.3+e1-6302~38~ubuntu16.04.1-stable)
+(kicad_pcb (version 4) (host pcbnew 4.0.4+e1-6308~48~ubuntu16.04.1-stable)
   (general
     (links 160)
@@
     (46 B.CrtYd user)
     (47 F.CrtYd user)
-    (48 B.Fab user)
-    (49 F.Fab user)
+    (48 B.Fab user hide)
+    (49 F.Fab user hide)
   )
   (setup
@@
     (effects (font (size 0.9 0.9) (thickness 0.2)) (justify mirror))
   )
-  (gr_text "RTC 36KHz" (at 123.53 45.72 90) (layer B.SilkS)
+  (gr_text "RTC 32KHz" (at 123.53 45.72 90) (layer B.SilkS)
     (effects (font (size 0.5 0.5) (thickness 0.125)) (justify mirror))
   )

Commit message: Some minor adjustment for pos file generation.
Parts:
- L1: value Ferr -> 600 Ferrite
- SW1: value TACT_G -> TACT
Changed lines of the file:
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@@
     (links 160)
     (no_connects 0)
-    (area 90.397667 29.02 150.215715 59.464)
+    (area 100.279999 36.769999 138.480001 54.670001)
     (thickness 1.6)
     (drawings 336)
@@
     (pad_drill 0.9652)
     (pad_to_mask_clearance 0.05)
-    (aux_axis_origin 0 0)
+    (aux_axis_origin 100.33 54.62)
     (grid_origin 100.33 45.72)
     (visible_elements FFFCFF7F)
@@
     (descr "Jumper SMD 0603, reflow soldering")
     (tags "jumper 0603")
-    (attr smd)
     (fp_text reference J1 (at 0 1.1) (layer B.Fab) hide
       (effects (font (size 0.635 0.635) (thickness 0.1)) (justify mirror))
@@
       (effects (font (size 0.635 0.635) (thickness 0.1)))
     )
-    (fp_text value Ferr (at 0 0) (layer F.Fab)
+    (fp_text value "600 Ferrite" (at 0 0) (layer F.Fab)
       (effects (font (size 0.635 0.635) (thickness 0.1)))
     )
@@
   (module pkl_connectors:Connector_USB_Micro_B_SMD (layer F.Cu)
     (at 101.755 45.72 180)
+    (attr smd)
     (fp_text reference P24 (at 0.025 0 270) (layer F.Fab)
       (effects (font (size 1 1) (thickness 0.15)))
@@
   (module pkl_misc:ABM8 (layer F.Cu)
     (at 130.63 48.02)
+    (attr smd)
     (fp_text reference X2 (at 0 0.7) (layer F.Fab)
       (effects (font (size 1 1) (thickness 0.15)))
@@
   (module pkl_samtec:FTSH-105-XX-X-DV (layer F.Cu)
     (at 111.53 45.72 90)
+    (attr smd)
     (fp_text reference X3 (at 0 1.3 90) (layer F.Fab)
       (effects (font (size 1 1) (thickness 0.15)))
@@
   (module pkl_buttons_switches:Tact_Switch_Top_B3U-1000P (layer F.Cu)
     (at 130.13 45.12 270)
+    (attr smd)
     (fp_text reference SW1 (at 0.45 0 360) (layer F.Fab)
       (effects (font (size 0.635 0.635) (thickness 0.15)))
     )
-    (fp_text value TACT_G (at -0.45 0 360) (layer F.Fab)
+    (fp_text value TACT (at -0.45 0 360) (layer F.Fab)
       (effects (font (size 0.635 0.635) (thickness 0.125)))
     )
@@
     (descr "Capacitor SMD 0603, reflow soldering")
     (tags "capacitor 0603")
-    (attr smd)
     (fp_text reference C6 (at 0 1.15 270) (layer B.Fab)
       (effects (font (size 0.635 0.635) (thickness 0.1)) (justify mirror))
@@
     (descr "Capacitor SMD 0603, reflow soldering")
     (tags "capacitor 0603")
-    (attr smd)
     (fp_text reference C7 (at 0 -1.2 90) (layer B.Fab)
       (effects (font (size 0.635 0.635) (thickness 0.1)) (justify mirror))
