File: 1bitsy/v1.0d/1bitsy.sch (KiCad schematic (older format))
At the start: 89 parts, among them J1 BOOT, P1 CONN_01X01, P10 CONN_01X01, P11 CONN_01X01, P12 CONN_01X01, P13 CONN_01X01, P14 CONN_01X01, P15 CONN_01X01, P16 CONN_01X01, P17 CONN_01X01, P18 CONN_01X01, P19 CONN_01X01, P2 CONN_01X01, P20 CONN_01X01, P21 CONN_01X01, P22 CONN_01X01, P23 CONN_01X01, P24 USB_OTG, P25 CONN_01X01, P26 CONN_01X01, P27 CONN_01X01, P28 CONN_01X01, P29 CONN_01X01, P3 CONN_01X01, P30 CONN_01X01, P31 CONN_01X01, P32 CONN_01X01, P33 CONN_01X01, P34 CONN_01X01, P35 CONN_01X01, P36 CONN_01X01, P37 CONN_01X01, P38 CONN_01X01, P39 CONN_01X01, P4 CONN_01X01, P40 CONN_01X01, P41 CONN_01X01, P42 CONN_01X01, P43 TP, P44 TP, P45 TP, P46 TP, P47 TP, P48 CONN_01X01, P49 CONN_01X01, P5 CONN_01X01, P50 CONN_01X01, P51 CONN_01X01, P52 CONN_01X01, P53 CONN_01X01, P54 CONN_01X01, P55 CONN_01X01, P6 CONN_01X01, P7 CONN_01X01, P8 CONN_01X01, P9 CONN_01X01, SW1 TACT_G, U1 VREG_3V3, U2 STM32F415RGT, X1 32.768kHz, X2 25MHz, X3 JTAG-10

Commit message: Some minor adjustment for pos file generation.
Parts:
- SW1: value TACT_G -> TACT; symbol TACT_G -> TACT; Key sw-tact-side-boss-gnd-3.0-2.5 -> sw-tact-top-30-25
Connections:
- net GND: no longer SW1.GND (case)
Changed lines of the file:
@@
 LIBS:pkl_texas
 LIBS:stm32
+LIBS:1bitsy
 LIBS:1bitsy-cache
 EELAYER 25 0
@@
 $EndDescr
 $Comp
-L GND #PWR6
+L GND #PWR01
 U 1 1 5743625A
 P 2350 9550
-F 0 "#PWR6" H 2350 9300 50  0001 C CNN
+F 0 "#PWR01" H 2350 9300 50  0001 C CNN
 F 1 "GND" H 2350 9400 50  0000 C CNN
 F 2 "" H 2350 9550 60  0000 C CNN
@@
 $EndComp
 $Comp
-L +3V3 #PWR1
+L +3V3 #PWR02
 U 1 1 5743625D
 P 650 8550
-F 0 "#PWR1" H 650 8400 50  0001 C CNN
+F 0 "#PWR02" H 650 8400 50  0001 C CNN
 F 1 "+3V3" H 650 8690 50  0000 C CNN
 F 2 "" H 650 8550 60  0000 C CNN
@@
 $EndComp
 $Comp
-L GND #PWR16
+L GND #PWR03
 U 1 1 5743625F
 P 13550 9250
-F 0 "#PWR16" H 13550 9000 50  0001 C CNN
+F 0 "#PWR03" H 13550 9000 50  0001 C CNN
 F 1 "GND" H 13550 9100 50  0000 C CNN
 F 2 "" H 13550 9250 60  0000 C CNN
@@
 $EndComp
 $Comp
-L GND #PWR4
+L GND #PWR04
 U 1 1 57436268
 P 1650 9550
-F 0 "#PWR4" H 1650 9300 50  0001 C CNN
+F 0 "#PWR04" H 1650 9300 50  0001 C CNN
 F 1 "GND" H 1650 9400 50  0000 C CNN
 F 2 "" H 1650 9550 60  0000 C CNN
@@
 $EndComp
 $Comp
-L GND #PWR17
+L GND #PWR05
 U 1 1 5743626B
 P 13850 9250
-F 0 "#PWR17" H 13850 9000 50  0001 C CNN
+F 0 "#PWR05" H 13850 9000 50  0001 C CNN
 F 1 "GND" H 13850 9100 50  0000 C CNN
 F 2 "" H 13850 9250 60  0000 C CNN
@@
 $EndComp
 $Comp
-L GND #PWR19
+L GND #PWR06
 U 1 1 5743626D
 P 14400 9250
-F 0 "#PWR19" H 14400 9000 50  0001 C CNN
+F 0 "#PWR06" H 14400 9000 50  0001 C CNN
 F 1 "GND" H 14400 9100 50  0000 C CNN
 F 2 "" H 14400 9250 60  0000 C CNN
@@
 $EndComp
 $Comp
-L GND #PWR18
+L GND #PWR07
 U 1 1 5743626F
 P 14150 9250
-F 0 "#PWR18" H 14150 9000 50  0001 C CNN
+F 0 "#PWR07" H 14150 9000 50  0001 C CNN
 F 1 "GND" H 14150 9100 50  0000 C CNN
 F 2 "" H 14150 9250 60  0000 C CNN
@@
 $EndComp
 $Comp
-L GND #PWR15
+L GND #PWR08
 U 1 1 57436271
 P 13550 6750
-F 0 "#PWR15" H 13550 6500 50  0001 C CNN
+F 0 "#PWR08" H 13550 6500 50  0001 C CNN
 F 1 "GND" H 13550 6600 50  0000 C CNN
 F 2 "" H 13550 6750 60  0000 C CNN
@@
 PC3
 $Comp
-L TACT_G SW1
+L TACT SW1
 U 1 1 57436285
 P 11000 1500
 F 0 "SW1" H 11150 1425 60  0000 L CNN
-F 1 "TACT_G" H 11150 1575 60  0000 L CNN
+F 1 "TACT" H 11150 1575 60  0000 L CNN
 F 2 "pkl_buttons_switches:Tact_Switch_Top_B3U-1000P" H 11000 1475 60  0001 C CNN
 F 3 "" H 11000 1475 60  0000 C CNN
-F 4 "sw-tact-side-boss-gnd-3.0-2.5" H 11000 1500 60  0001 C CNN "Key"
+F 4 "sw-tact-top-30-25" H 11000 1500 60  0001 C CNN "Key"
 F 5 "B3U-1000P" H 11000 1500 60  0001 C CNN "MFN"
 F 6 "ANY" H 11000 1500 60  0001 C CNN "Source"
@@
 $EndComp
 $Comp
-L GND #PWR13
+L GND #PWR09
 U 1 1 57436286
 P 10700 1900
-F 0 "#PWR13" H 10700 1650 50  0001 C CNN
+F 0 "#PWR09" H 10700 1650 50  0001 C CNN
 F 1 "GND" H 10700 1750 50  0000 C CNN
 F 2 "" H 10700 1900 60  0000 C CNN
@@
 BUTTON
 $Comp
-L +3V3 #PWR14
+L +3V3 #PWR010
 U 1 1 57436288
 P 11500 1100
-F 0 "#PWR14" H 11500 950 50  0001 C CNN
+F 0 "#PWR010" H 11500 950 50  0001 C CNN
 F 1 "+3V3" H 11500 1240 50  0000 C CNN
 F 2 "" H 11500 1100 60  0000 C CNN
@@
 ~RST
 $Comp
-L GND #PWR9
+L GND #PWR011
 U 1 1 5743628B
 P 3150 4250
-F 0 "#PWR9" H 3150 4000 50  0001 C CNN
+F 0 "#PWR011" H 3150 4000 50  0001 C CNN
 F 1 "GND" H 3150 4100 50  0000 C CNN
 F 2 "" H 3150 4250 60  0000 C CNN
@@
 $EndComp
 $Comp
-L +3V3 #PWR8
+L +3V3 #PWR012
 U 1 1 5743628C
 P 3150 3650
-F 0 "#PWR8" H 3150 3500 50  0001 C CNN
+F 0 "#PWR012" H 3150 3500 50  0001 C CNN
 F 1 "+3V3" H 3150 3790 50  0000 C CNN
 F 2 "" H 3150 3650 60  0000 C CNN
@@
 $EndComp
 $Comp
-L GND #PWR10
+L GND #PWR013
 U 1 1 5743628E
 P 4350 1800
-F 0 "#PWR10" H 4350 1550 50  0001 C CNN
+F 0 "#PWR013" H 4350 1550 50  0001 C CNN
 F 1 "GND" H 4350 1650 50  0000 C CNN
 F 2 "" H 4350 1800 60  0000 C CNN
@@
 $EndComp
 $Comp
-L GND #PWR11
+L GND #PWR014
 U 1 1 57436290
 P 4950 1800
-F 0 "#PWR11" H 4950 1550 50  0001 C CNN
+F 0 "#PWR014" H 4950 1550 50  0001 C CNN
 F 1 "GND" H 4950 1650 50  0000 C CNN
 F 2 "" H 4950 1800 60  0000 C CNN
@@
 $EndComp
 $Comp
-L +3V3 #PWR12
+L +3V3 #PWR015
 U 1 1 574362A9
 P 9750 1250
-F 0 "#PWR12" H 9750 1100 50  0001 C CNN
+F 0 "#PWR015" H 9750 1100 50  0001 C CNN
 F 1 "+3V3" H 9750 1390 50  0000 C CNN
 F 2 "" H 9750 1250 60  0000 C CNN
@@
 $EndComp
 $Comp
-L PWR_FLAG #FLG1
+L PWR_FLAG #FLG016
 U 1 1 574362B9
 P 1050 8600
-F 0 "#FLG1" H 1050 8695 50  0001 C CNN
+F 0 "#FLG016" H 1050 8695 50  0001 C CNN
 F 1 "PWR_FLAG" H 1050 8780 50  0000 C CNN
 F 2 "" H 1050 8600 60  0000 C CNN
@@
 $EndComp
 $Comp
-L PWR_FLAG #FLG3
+L PWR_FLAG #FLG017
 U 1 1 574362BA
 P 13750 7650
-F 0 "#FLG3" H 13750 7745 50  0001 C CNN
+F 0 "#FLG017" H 13750 7745 50  0001 C CNN
 F 1 "PWR_FLAG" H 13750 7830 50  0000 C CNN
 F 2 "" H 13750 7650 60  0000 C CNN
@@
 $EndComp
 $Comp
-L PWR_FLAG #FLG4
+L PWR_FLAG #FLG018
 U 1 1 574362BB
 P 13950 7450
-F 0 "#FLG4" H 13950 7545 50  0001 C CNN
+F 0 "#FLG018" H 13950 7545 50  0001 C CNN
 F 1 "PWR_FLAG" H 13950 7630 50  0000 C CNN
 F 2 "" H 13950 7450 60  0000 C CNN
@@
 	2050 7450 2450 7450
 Wire Wire Line
-	11000 1700 11000 1800
-Wire Wire Line
 	10800 1500 10700 1500
 Wire Wire Line
 	11200 1500 11700 1500
-Wire Wire Line
-	10700 1500 10700 1900
-Wire Wire Line
-	11000 1800 10700 1800
-Connection ~ 10700 1800
 Wire Wire Line
 	11500 1500 11500 1400
@@
 $EndComp
 $Comp
-L GND #PWR5
+L GND #PWR019
 U 1 1 574438ED
 P 2300 1750
-F 0 "#PWR5" H 2300 1500 50  0001 C CNN
+F 0 "#PWR019" H 2300 1500 50  0001 C CNN
 F 1 "GND" H 2300 1600 50  0000 C CNN
 F 2 "" H 2300 1750 60  0000 C CNN
@@
 $EndComp
 $Comp
-L +3V3 #PWR7
+L +3V3 #PWR020
 U 1 1 574438EF
 P 2700 1050
-F 0 "#PWR7" H 2700 900 50  0001 C CNN
+F 0 "#PWR020" H 2700 900 50  0001 C CNN
 F 1 "+3V3" H 2700 1190 50  0000 C CNN
 F 2 "" H 2700 1050 60  0000 C CNN
@@
 $EndComp
 $Comp
-L PWR_FLAG #FLG2
+L PWR_FLAG #FLG021
 U 1 1 574438F1
 P 1500 1050
-F 0 "#FLG2" H 1500 1145 50  0001 C CNN
+F 0 "#FLG021" H 1500 1145 50  0001 C CNN
 F 1 "PWR_FLAG" H 1500 1230 50  0000 C CNN
 F 2 "" H 1500 1050 60  0000 C CNN
@@
 	2600 1350 2700 1350
 Wire Wire Line
-	2700 1650 2700 1350
+	2700 1350 2700 1650
 Wire Wire Line
 	1500 1650 2900 1650
@@
 $EndComp
 $Comp
-L GND #PWR3
+L GND #PWR022
 U 1 1 574838B5
 P 1100 1650
-F 0 "#PWR3" H 1100 1400 50  0001 C CNN
+F 0 "#PWR022" H 1100 1400 50  0001 C CNN
 F 1 "GND" H 1100 1500 50  0000 C CNN
 F 2 "" H 1100 1650 60  0000 C CNN
@@
 	1100 1050 1100 1250
 $Comp
-L +3V3 #PWR2
+L +3V3 #PWR023
 U 1 1 5751C607
 P 1100 1050
-F 0 "#PWR2" H 1100 900 50  0001 C CNN
+F 0 "#PWR023" H 1100 900 50  0001 C CNN
 F 1 "+3V3" H 1100 1190 50  0000 C CNN
 F 2 "" H 1100 1050 60  0000 C CNN
@@
 Text Label 13750 6350 0    60   ~ 0
 PD2
+Wire Wire Line
+	10700 1500 10700 1900
 $EndSCHEMATC
